Commit message: description: add 'khi_' prefix to macro name.
To avoid name clashes with other macros that happen to have the same name.

File: duaro_description/urdf/duaro.urdf.xacro (robot description, xacro)
@@ -1,7 +1,7 @@
 <?xml version="1.0" ?>
-<robot name="duaro" xmlns:xacro="http://ros.org/wiki/xacro">
+<robot name="khi_duaro" xmlns:xacro="http://ros.org/wiki/xacro">
   <xacro:include filename="$(find duaro_description)/urdf/duaro_macro.xacro"/>
   <!-- instantiate duaro -->
-  <xacro:duaro />
+  <xacro:khi_duaro />
   <!-- Fix duaro to world -->
   <link name="world"/>

File: duaro_description/urdf/duaro_macro.xacro (robot description, xacro)
@@ -1,5 +1,5 @@
 <?xml version="1.0"?>
 <robot xmlns:xacro="http://ros.org/wiki/xacro">
-  <xacro:macro name="duaro">
+  <xacro:macro name="khi_duaro">
     <xacro:include filename="$(find duaro_description)/urdf/duaro.transmission.xacro" />
     <!-- DH params -->

File: rs_description/urdf/rs007l.urdf.xacro (robot description, xacro)
@@ -1,7 +1,7 @@
 <?xml version="1.0" ?>
-<robot name="rs007l" xmlns:xacro="http://ros.org/wiki/xacro">
+<robot name="khi_rs007l" xmlns:xacro="http://ros.org/wiki/xacro">
   <xacro:include filename="$(find rs_description)/urdf/rs007l_macro.xacro"/>
   <!-- instantiate rs007l -->
-  <xacro:rs007l />
+  <xacro:khi_rs007l />
   <!-- Fix rs007l to world -->
   <link name="world"/>

File: rs_description/urdf/rs007l_macro.xacro (robot description, xacro)
@@ -1,5 +1,5 @@
 <?xml version="1.0"?>
 <robot xmlns:xacro="http://ros.org/wiki/xacro">
-  <xacro:macro name="rs007l">
+  <xacro:macro name="khi_rs007l">
     <xacro:include filename="$(find rs_description)/urdf/rs.transmission.xacro" />
     <xacro:include filename="$(find rs_description)/urdf/common.gazebo.xacro" />

File: rs_description/urdf/rs007n.urdf.xacro (robot description, xacro)
@@ -1,7 +1,7 @@
 <?xml version="1.0" ?>
-<robot name="rs007n" xmlns:xacro="http://ros.org/wiki/xacro">
+<robot name="khi_rs007n" xmlns:xacro="http://ros.org/wiki/xacro">
   <xacro:include filename="$(find rs_description)/urdf/rs007n_macro.xacro"/>
   <!-- instantiate rs007n -->
-  <xacro:rs007n />
+  <xacro:khi_rs007n />
   <!-- Fix rs007n to world -->
   <link name="world"/>

File: rs_description/urdf/rs007n_macro.xacro (robot description, xacro)
@@ -1,5 +1,5 @@
 <?xml version="1.0"?>
 <robot xmlns:xacro="http://ros.org/wiki/xacro">
-  <xacro:macro name="rs007n">
+  <xacro:macro name="khi_rs007n">
     <xacro:include filename="$(find rs_description)/urdf/rs.transmission.xacro" />
     <xacro:include filename="$(find rs_description)/urdf/common.gazebo.xacro" />

File: rs_description/urdf/rs080n.urdf.xacro (robot description, xacro)
@@ -1,7 +1,7 @@
 <?xml version="1.0" ?>
-<robot name="rs080n" xmlns:xacro="http://ros.org/wiki/xacro">
+<robot name="khi_rs080n" xmlns:xacro="http://ros.org/wiki/xacro">
   <xacro:include filename="$(find rs_description)/urdf/rs080n_macro.xacro"/>
   <!-- instantiate rs080n -->
-  <xacro:rs080n />
+  <xacro:khi_rs080n />
   <!-- Fix rs080n to world -->
   <link name="world"/>

File: rs_description/urdf/rs080n_macro.xacro (robot description, xacro)
@@ -1,5 +1,5 @@
 <?xml version="1.0"?>
 <robot xmlns:xacro="http://ros.org/wiki/xacro">
-  <xacro:macro name="rs080n">
+  <xacro:macro name="khi_rs080n">
     <xacro:include filename="$(find rs_description)/urdf/rs.transmission.xacro" />
     <xacro:include filename="$(find rs_description)/urdf/common.gazebo.xacro" />
