Commit message: description: add 'prefix' arg to xacro macro.
Allows for prepending a prefix to the name of links and joints, to avoid name clashes between links and joints from other xacro macros in a composite xacro.

File: duaro_description/urdf/duaro.urdf.xacro (robot description, xacro)
@@ -3,5 +3,5 @@
   <xacro:include filename="$(find duaro_description)/urdf/duaro_macro.xacro"/>
   <!-- instantiate duaro -->
-  <xacro:khi_duaro />
+  <xacro:khi_duaro prefix="" />
   <!-- Fix duaro to world -->
   <link name="world"/>

File: duaro_description/urdf/duaro_macro.xacro (robot description, xacro)
@@ -1,5 +1,5 @@
 <?xml version="1.0"?>
 <robot xmlns:xacro="http://ros.org/wiki/xacro">
-  <xacro:macro name="khi_duaro">
+  <xacro:macro name="khi_duaro" params="prefix">
     <xacro:include filename="$(find duaro_description)/urdf/duaro.transmission.xacro" />
     <!-- DH params -->
@@ -68,5 +68,5 @@
       </inertial>
     </xacro:macro>
-    <link name="base_link">
+    <link name="${prefix}base_link">
       <visual>
         <geometry>
@@ -85,6 +85,6 @@
     </link>
     <!-- fixed parts xacro-->
-    <xacro:macro name="fixed_parts" params="color name height rot mass">
-      <link name="${name}">
+    <xacro:macro name="fixed_parts" params="prefix:=^ color name height rot mass">
+      <link name="${prefix}${name}">
         <visual>
           <geometry>
@@ -102,7 +102,7 @@
         <xacro:default_inertial mass="${mass}"/>
       </link>
-      <joint name="${name}_joint" type="fixed">
-        <parent link="base_link"/>
-        <child link="${name}"/>
+      <joint name="${prefix}${name}_joint" type="fixed">
+        <parent link="${prefix}base_link"/>
+        <child link="${prefix}${name}"/>
         <origin xyz="0 0 ${height}" rpy="0 0 0" />
       </joint>
@@ -113,5 +113,5 @@
     <xacro:fixed_parts color="Black" name="duaro_logo" height="0" rot="${pi/2}" mass="1"/>
     <xacro:fixed_parts color="Light_blue" name="pedestal_obstacle" height="0" rot="0" mass="2"/>
-    <link name="duaro_j0">
+    <link name="${prefix}duaro_j0">
       <visual>
         <geometry>
@@ -129,11 +129,11 @@
       <xacro:default_inertial mass="10"/>
     </link>
-    <joint name="joint0" type="fixed">
+    <joint name="${prefix}joint0" type="fixed">
       <origin xyz="0 0 0.82"/>
-      <parent link="duaro_body"/>
-      <child link="duaro_j0"/>
+      <parent link="${prefix}duaro_body"/>
+      <child link="${prefix}duaro_j0"/>
     </joint>
     <!-- lower arm -->
-    <link name="lower_link_j1">
+    <link name="${prefix}lower_link_j1">
       <visual>
         <geometry>
@@ -152,13 +152,13 @@
       <xacro:link_inertial Izz="${L1_Izz}" length="${L1_length}" mass="${L1_mass}"/>
     </link>
-    <joint name="lower_joint1" type="revolute">
+    <joint name="${prefix}lower_joint1" type="revolute">
         <axis xyz="0 0 1" rpy="0 0 0" />
         <limit effort="100.0" lower="${J1_LOWER_lower_limit}" upper="${J1_LOWER_upper_limit}" velocity="${J1_velocity_limit}"/>
         <origin xyz="0 0 0.2515" rpy="0 0 0"/>
-        <parent link="duaro_j0"/>
-        <child link="lower_link_j1"/>
+        <parent link="${prefix}duaro_j0"/>
+        <child link="${prefix}lower_link_j1"/>
         <dynamics damping="0.0" friction="0.0"/>
     </joint>
-    <link name="lower_link_j2">
+    <link name="${prefix}lower_link_j2">
       <visual>
         <geometry>
@@ -177,13 +177,13 @@
       <xacro:link_inertial Izz="${L2_Izz}" length="${L2_length}" mass="${L2_mass}"/>
     </link>
-    <joint name="lower_joint2" type="revolute">
+    <joint name="${prefix}lower_joint2" type="revolute">
       <axis xyz="0 0 1" rpy="0 0 0" />
       <limit effort="100.0" lower="${J2_LOWER_lower_limit}" upper="${J2_LOWER_upper_limit}" velocity="${J2_velocity_limit}"/>
       <origin xyz="0 ${dh_j1_j2_transy} 0.0905"/>
-      <parent link="lower_link_j1"/>
-      <child link="lower_link_j2"/>
+      <parent link="${prefix}lower_link_j1"/>
+      <child link="${prefix}lower_link_j2"/>
       <dynamics damping="0.0" friction="0.0"/>
     </joint>
-    <link name="lower_link_j3">
+    <link name="${prefix}lower_link_j3">
       <visual>
         <geometry>
@@ -202,12 +202,12 @@
       <xacro:default_inertial mass="${L3_mass}"/>
     </link>
-    <joint name="lower_joint3" type="prismatic">
+    <joint name="${prefix}lower_joint3" type="prismatic">
       <axis xyz="0 0 1" rpy="0 0 0" />
       <limit effort="100.0" lower="${J3_LOWER_lower_limit}" upper="${J3_LOWER_upper_limit}" velocity="${J3_velocity_limit}"/>
       <origin xyz="0 ${dh_j2_j3_transy} 0.03850"/>
-      <parent link="lower_link_j2"/>
-      <child link="lower_link_j3"/>
-    </joint>
-    <link name="lower_link_j3_obst">
+      <parent link="${prefix}lower_link_j2"/>
+      <child link="${prefix}lower_link_j3"/>
+    </joint>
+    <link name="${prefix}lower_link_j3_obst">
       <visual>
         <geometry>
@@ -218,10 +218,10 @@
       </visual>
     </link>
-    <joint name="lower_j3_obstaclem_joint" type="fixed">
+    <joint name="${prefix}lower_j3_obstaclem_joint" type="fixed">
       <origin rpy="0 0 0" xyz="0 0 0"/>
-      <parent link="lower_link_j3"/>
-      <child link="lower_link_j3_obst"/>
-    </joint>
-    <link name="lower_link_j4">
+      <parent link="${prefix}lower_link_j3"/>
+      <child link="${prefix}lower_link_j3_obst"/>
+    </joint>
+    <link name="${prefix}lower_link_j4">
       <visual>
         <geometry>
@@ -240,14 +240,14 @@
       <xacro:default_inertial mass="0.5"/>
     </link>
-    <joint name="lower_joint4" type="revolute">
+    <joint name="${prefix}lower_joint4" type="revolute">
       <axis xyz="0 0 1" rpy="0 0 0" />
       <limit effort="100.0" lower="${J4_LOWER_lower_limit}" upper="${J4_LOWER_upper_limit}" velocity="${J4_velocity_limit}"/>
       <origin xyz="0 0 -0.24"/>
-      <parent link="lower_link_j3"/>
-      <child link="lower_link_j4"/>
+      <parent link="${prefix}lower_link_j3"/>
+      <child link="${prefix}lower_link_j4"/>
       <dynamics damping="0.0" friction="0.0"/>
     </joint>
     <!-- upper arm -->
-    <link name="upper_link_j1">
+    <link name="${prefix}upper_link_j1">
       <visual>
         <geometry>
@@ -266,13 +266,13 @@
       <xacro:link_inertial Izz="${U1_Izz}" length="${U1_length}" mass="${U1_mass}"/>
     </link>
-    <joint name="upper_joint1" type="revolute">
+    <joint name="${prefix}upper_joint1" type="revolute">
       <origin rpy="0 0 0" xyz="0 0 0.3805"/>
         <axis xyz="0 0 1" rpy="0 0 0" />
         <limit effort="100.0" lower="${J1_UPPER_lower_limit}" upper="${J1_UPPER_upper_limit}" velocity="${J1_velocity_limit}"/>
-        <parent link="duaro_j0"/>
-        <child link="upper_link_j1"/>
+        <parent link="${prefix}duaro_j0"/>
+        <child link="${prefix}upper_link_j1"/>
         <dynamics damping="0.0" friction="0.0"/>
     </joint>
-    <link name="upper_link_j2">
+    <link name="${prefix}upper_link_j2">
       <visual>
         <geometry>
@@ -291,13 +291,13 @@
       <xacro:link_inertial Izz="${U2_Izz}" length="${U2_length}" mass="${U2_mass}"/>
     </link>
-    <joint name="upper_joint2" type="revolute">
+    <joint name="${prefix}upper_joint2" type="revolute">
       <axis xyz="0 0 1" rpy="0 0 0" />
       <limit effort="100.0" lower="${J2_UPPER_lower_limit}" upper="${J2_UPPER_upper_limit}" velocity="${J2_velocity_limit}"/>
       <origin xyz="0 ${dh_j1_j2_transy} 0"/>
-      <parent link="upper_link_j1"/>
-      <child link="upper_link_j2"/>
+      <parent link="${prefix}upper_link_j1"/>
+      <child link="${prefix}upper_link_j2"/>
       <dynamics damping="0.0" friction="0.0"/>
     </joint>
-    <link name="upper_link_j3">
+    <link name="${prefix}upper_link_j3">
       <visual>
         <geometry>
@@ -316,12 +316,12 @@
       <xacro:default_inertial mass="${U3_mass}"/>
     </link>
-    <joint name="upper_joint3" type="prismatic">
+    <joint name="${prefix}upper_joint3" type="prismatic">
       <axis xyz="0 0 1" rpy="0 0 0" />
       <limit effort="100.0" lower="${J3_UPPER_lower_limit}" upper="${J3_UPPER_upper_limit}" velocity="${J3_velocity_limit}"/>
       <origin xyz="0 ${dh_j2_j3_transy} 0"/>
-      <parent link="upper_link_j2"/>
-      <child link="upper_link_j3"/>
-    </joint>
-    <link name="upper_link_j3_obst">
+      <parent link="${prefix}upper_link_j2"/>
+      <child link="${prefix}upper_link_j3"/>
+    </joint>
+    <link name="${prefix}upper_link_j3_obst">
       <visual>
         <geometry>
@@ -332,10 +332,10 @@
       </visual>
     </link>
-    <joint name="upper_j3_obstaclem_joint" type="fixed">
+    <joint name="${prefix}upper_j3_obstaclem_joint" type="fixed">
       <origin xyz="0 0 0"/>
-      <parent link="upper_link_j3"/>
-      <child link="upper_link_j3_obst"/>
-    </joint>
-   <link name="upper_link_j4">
+      <parent link="${prefix}upper_link_j3"/>
+      <child link="${prefix}upper_link_j3_obst"/>
+    </joint>
+   <link name="${prefix}upper_link_j4">
       <visual>
         <geometry>
@@ -354,10 +354,10 @@
       <xacro:default_inertial mass="10"/>
     </link>
-    <joint name="upper_joint4" type="revolute">
+    <joint name="${prefix}upper_joint4" type="revolute">
       <axis xyz="0 0 1" rpy="0 0 0" />
       <limit effort="100.0" lower="${J4_UPPER_lower_limit}" upper="${J4_UPPER_upper_limit}" velocity="${J3_velocity_limit}"/>
       <origin xyz="0 0 -0.24"/>
-      <parent link="upper_link_j3"/>
-      <child link="upper_link_j4"/>
+      <parent link="${prefix}upper_link_j3"/>
+      <child link="${prefix}upper_link_j4"/>
       <dynamics damping="0.0" friction="0.0"/>
     </joint>
@@ -368,21 +368,21 @@
     </gazebo>
     </xacro:macro>
-    <xacro:gazebo_color parts="duaro_body" colors="White"/>
-    <xacro:gazebo_color parts="pedestal_obstacle" colors="Light_blue"/>
-    <xacro:gazebo_color parts="duaro_logo" colors="Black"/>
-    <xacro:gazebo_color parts="base_link" colors="White"/>
-    <xacro:gazebo_color parts="duaro_j0" colors="White"/>
-    <xacro:gazebo_color parts="duaro_j0_cover" colors="Light_blue"/>
-    <xacro:gazebo_color parts="lower_link_j1" colors="White"/>
-    <xacro:gazebo_color parts="lower_link_j2" colors="White"/>
-    <xacro:gazebo_color parts="lower_link_j3" colors="White"/>
-    <xacro:gazebo_color parts="lower_link_j4" colors="White"/>
-    <xacro:gazebo_color parts="lower_link_j3_obst" colors="Black"/>
-    <xacro:gazebo_color parts="upper_link_j1" colors="White"/>
-    <xacro:gazebo_color parts="upper_link_j2" colors="White"/>
-    <xacro:gazebo_color parts="upper_link_j3" colors="White"/>
-    <xacro:gazebo_color parts="upper_link_j4" colors="White"/>
-    <xacro:gazebo_color parts="upper_link_j3_obst" colors="Black"/>
-    <xacro:gazebo_color parts="duaro_body" colors="White"/>
+    <xacro:gazebo_color parts="${prefix}duaro_body" colors="White"/>
+    <xacro:gazebo_color parts="${prefix}pedestal_obstacle" colors="Light_blue"/>
+    <xacro:gazebo_color parts="${prefix}duaro_logo" colors="Black"/>
+    <xacro:gazebo_color parts="${prefix}base_link" colors="White"/>
+    <xacro:gazebo_color parts="${prefix}duaro_j0" colors="White"/>
+    <xacro:gazebo_color parts="${prefix}duaro_j0_cover" colors="Light_blue"/>
+    <xacro:gazebo_color parts="${prefix}lower_link_j1" colors="White"/>
+    <xacro:gazebo_color parts="${prefix}lower_link_j2" colors="White"/>
+    <xacro:gazebo_color parts="${prefix}lower_link_j3" colors="White"/>
+    <xacro:gazebo_color parts="${prefix}lower_link_j4" colors="White"/>
+    <xacro:gazebo_color parts="${prefix}lower_link_j3_obst" colors="Black"/>
+    <xacro:gazebo_color parts="${prefix}upper_link_j1" colors="White"/>
+    <xacro:gazebo_color parts="${prefix}upper_link_j2" colors="White"/>
+    <xacro:gazebo_color parts="${prefix}upper_link_j3" colors="White"/>
+    <xacro:gazebo_color parts="${prefix}upper_link_j4" colors="White"/>
+    <xacro:gazebo_color parts="${prefix}upper_link_j3_obst" colors="Black"/>
+    <xacro:gazebo_color parts="${prefix}duaro_body" colors="White"/>
     <!-- duaro end -->
     <gazebo>

File: rs_description/urdf/rs007l.urdf.xacro (robot description, xacro)
@@ -3,5 +3,5 @@
   <xacro:include filename="$(find rs_description)/urdf/rs007l_macro.xacro"/>
   <!-- instantiate rs007l -->
-  <xacro:khi_rs007l />
+  <xacro:khi_rs007l prefix="" />
   <!-- Fix rs007l to world -->
   <link name="world"/>

File: rs_description/urdf/rs007l_macro.xacro (robot description, xacro)
@@ -1,5 +1,5 @@
 <?xml version="1.0"?>
 <robot xmlns:xacro="http://ros.org/wiki/xacro">
-  <xacro:macro name="khi_rs007l">
+  <xacro:macro name="khi_rs007l" params="prefix">
     <xacro:include filename="$(find rs_description)/urdf/rs.transmission.xacro" />
     <xacro:include filename="$(find rs_description)/urdf/common.gazebo.xacro" />
@@ -60,5 +60,5 @@
     <!-- rs007l start -->
     <!-- Link 0 -->
-    <link name="base_link">
+    <link name="${prefix}base_link">
       <visual>
         <geometry>
@@ -78,13 +78,13 @@
     </link>
     <!-- Link 1 -->
-    <joint name="joint1" type="revolute">
+    <joint name="${prefix}joint1" type="revolute">
       <axis xyz="0 0 -1" rpy="0 0 0" />
       <limit effort="1000.0" lower="${j1_lower_limit}" upper="${j1_upper_limit}" velocity="${j1_velocity_limit}"/>
       <origin xyz="0 0 ${j0_length}" rpy="0 0 0" />
-      <parent link="base_link"/>
-      <child link="link1"/>
-      <dynamics damping="0.0" friction="0.0"/>
-    </joint>
-    <link name="link1">
+      <parent link="${prefix}base_link"/>
+      <child link="${prefix}link1"/>
+      <dynamics damping="0.0" friction="0.0"/>
+    </joint>
+    <link name="${prefix}link1">
       <visual>
         <geometry>
@@ -104,13 +104,13 @@
     </link>
     <!-- Link 2 -->
-    <joint name="joint2" type="revolute">
+    <joint name="${prefix}joint2" type="revolute">
       <axis xyz="0 0 1" rpy="0 0 0" />
       <limit effort="1000.0" lower="${j2_lower_limit}" upper="${j2_upper_limit}" velocity="${j2_velocity_limit}"/>
       <origin xyz="0 0 ${j1_length}" rpy="0 ${dh_j1_j2_roty} 0" />
-      <parent link="link1"/>
-      <child link="link2"/>
-      <dynamics damping="0.0" friction="0.0"/>
-    </joint>
-    <link name="link2">
+      <parent link="${prefix}link1"/>
+      <child link="${prefix}link2"/>
+      <dynamics damping="0.0" friction="0.0"/>
+    </joint>
+    <link name="${prefix}link2">
       <visual>
         <geometry>
@@ -130,13 +130,13 @@
     </link>
     <!-- Link 3 -->
-    <joint name="joint3" type="revolute">
+    <joint name="${prefix}joint3" type="revolute">
       <axis xyz="0 0 -1" rpy="0 0 0" />
       <limit effort="1000.0" lower="${j3_lower_limit}" upper="${j3_upper_limit}" velocity="${j3_velocity_limit}"/>
       <origin xyz="${j2_length} 0 0" rpy="0 0 0" />
-      <parent link="link2"/>
-      <child link="link3"/>
-      <dynamics damping="0.0" friction="0.0"/>
-    </joint>
-    <link name="link3">
+      <parent link="${prefix}link2"/>
+      <child link="${prefix}link3"/>
+      <dynamics damping="0.0" friction="0.0"/>
+    </joint>
+    <link name="${prefix}link3">
       <visual>
         <geometry>
@@ -156,13 +156,13 @@
     </link>
     <!-- Link 4 -->
-    <joint name="joint4" type="revolute">
+    <joint name="${prefix}joint4" type="revolute">
       <axis xyz="0 0 1" rpy="0 0 0" />
       <limit effort="1000.0" lower="${j4_lower_limit}" upper="${j4_upper_limit}" velocity="${j4_velocity_limit}"/>
       <origin xyz="${j3_length} 0 0" rpy="0 ${dh_j3_j4_roty} 0" />
-      <parent link="link3"/>
-      <child link="link4"/>
-      <dynamics damping="0.0" friction="0.0"/>
-    </joint>
-    <link name="link4">
+      <parent link="${prefix}link3"/>
+      <child link="${prefix}link4"/>
+      <dynamics damping="0.0" friction="0.0"/>
+    </joint>
+    <link name="${prefix}link4">
       <visual>
         <geometry>
@@ -182,13 +182,13 @@
     </link>
     <!-- Link 5 -->
-    <joint name="joint5" type="revolute">
+    <joint name="${prefix}joint5" type="revolute">
       <axis xyz="0 0 -1" rpy="0 0 0" />
       <limit effort="1000.0" lower="${j5_lower_limit}" upper="${j5_upper_limit}" velocity="${j5_velocity_limit}"/>
       <origin xyz="0 0 ${j4_length}" rpy="0 ${dh_j4_j5_roty} 0" />
-      <parent link="link4"/>
-      <child link="link5"/>
-      <dynamics damping="0.0" friction="0.0"/>
-    </joint>
-    <link name="link5">
+      <parent link="${prefix}link4"/>
+      <child link="${prefix}link5"/>
+      <dynamics damping="0.0" friction="0.0"/>
+    </joint>
+    <link name="${prefix}link5">
       <visual>
         <geometry>
@@ -208,13 +208,13 @@
     </link>
     <!-- Link 6 -->
-    <joint name="joint6" type="revolute">
+    <joint name="${prefix}joint6" type="revolute">
       <axis xyz="0 0 1" rpy="0 0 0" />
       <limit effort="1000.0" lower="${j6_lower_limit}" upper="${j6_upper_limit}" velocity="${j6_velocity_limit}"/>
       <origin xyz="${j5_length} 0 0" rpy="0 ${dh_j5_j6_roty} 0" />
-      <parent link="link5"/>
-      <child link="link6"/>
-      <dynamics damping="0.0" friction="0.0"/>
-    </joint>
-    <link name="link6">
+      <parent link="${prefix}link5"/>
+      <child link="${prefix}link6"/>
+      <dynamics damping="0.0" friction="0.0"/>
+    </joint>
+    <link name="${prefix}link6">
       <visual>
         <geometry>

File: rs_description/urdf/rs007n.urdf.xacro (robot description, xacro)
@@ -3,5 +3,5 @@
   <xacro:include filename="$(find rs_description)/urdf/rs007n_macro.xacro"/>
   <!-- instantiate rs007n -->
-  <xacro:khi_rs007n />
+  <xacro:khi_rs007n prefix="" />
   <!-- Fix rs007n to world -->
   <link name="world"/>

File: rs_description/urdf/rs007n_macro.xacro (robot description, xacro)
@@ -1,5 +1,5 @@
 <?xml version="1.0"?>
 <robot xmlns:xacro="http://ros.org/wiki/xacro">
-  <xacro:macro name="khi_rs007n">
+  <xacro:macro name="khi_rs007n" params="prefix">
     <xacro:include filename="$(find rs_description)/urdf/rs.transmission.xacro" />
     <xacro:include filename="$(find rs_description)/urdf/common.gazebo.xacro" />
@@ -60,5 +60,5 @@
     <!-- rs007n start -->
     <!-- Link 0 -->
-    <link name="base_link">
+    <link name="${prefix}base_link">
       <visual>
         <geometry>
@@ -78,13 +78,13 @@
     </link>
     <!-- Link 1 -->
-    <joint name="joint1" type="revolute">
+    <joint name="${prefix}joint1" type="revolute">
       <axis xyz="0 0 -1" rpy="0 0 0" />
       <limit effort="1000.0" lower="${j1_lower_limit}" upper="${j1_upper_limit}" velocity="${j1_velocity_limit}"/>
       <origin xyz="0 0 ${j0_length}" rpy="0 0 0" />
-      <parent link="base_link"/>
-      <child link="link1"/>
-      <dynamics damping="0.0" friction="0.0"/>
-    </joint>
-    <link name="link1">
+      <parent link="${prefix}base_link"/>
+      <child link="${prefix}link1"/>
+      <dynamics damping="0.0" friction="0.0"/>
+    </joint>
+    <link name="${prefix}link1">
       <visual>
         <geometry>
@@ -104,13 +104,13 @@
     </link>
     <!-- Link 2 -->
-    <joint name="joint2" type="revolute">
+    <joint name="${prefix}joint2" type="revolute">
       <axis xyz="0 0 1" rpy="0 0 0" />
       <limit effort="1000.0" lower="${j2_lower_limit}" upper="${j2_upper_limit}" velocity="${j2_velocity_limit}"/>
       <origin xyz="0 0 ${j1_length}" rpy="0 ${dh_j1_j2_roty} 0" />
-      <parent link="link1"/>
-      <child link="link2"/>
-      <dynamics damping="0.0" friction="0.0"/>
-    </joint>
-    <link name="link2">
+      <parent link="${prefix}link1"/>
+      <child link="${prefix}link2"/>
+      <dynamics damping="0.0" friction="0.0"/>
+    </joint>
+    <link name="${prefix}link2">
       <visual>
         <geometry>
@@ -130,13 +130,13 @@
     </link>
     <!-- Link 3 -->
-    <joint name="joint3" type="revolute">
+    <joint name="${prefix}joint3" type="revolute">
       <axis xyz="0 0 -1" rpy="0 0 0" />
       <limit effort="1000.0" lower="${j3_lower_limit}" upper="${j3_upper_limit}" velocity="${j3_velocity_limit}"/>
       <origin xyz="${j2_length} 0 0" rpy="0 0 0" />
-      <parent link="link2"/>
-      <child link="link3"/>
-      <dynamics damping="0.0" friction="0.0"/>
-    </joint>
-    <link name="link3">
+      <parent link="${prefix}link2"/>
+      <child link="${prefix}link3"/>
+      <dynamics damping="0.0" friction="0.0"/>
+    </joint>
+    <link name="${prefix}link3">
       <visual>
         <geometry>
@@ -156,13 +156,13 @@
     </link>
     <!-- Link 4 -->
-    <joint name="joint4" type="revolute">
+    <joint name="${prefix}joint4" type="revolute">
       <axis xyz="0 0 1" rpy="0 0 0" />
       <limit effort="1000.0" lower="${j4_lower_limit}" upper="${j4_upper_limit}" velocity="${j4_velocity_limit}"/>
       <origin xyz="${j3_length} 0 0" rpy="0 ${dh_j3_j4_roty} 0" />
-      <parent link="link3"/>
-      <child link="link4"/>
-      <dynamics damping="0.0" friction="0.0"/>
-    </joint>
-    <link name="link4">
+      <parent link="${prefix}link3"/>
+      <child link="${prefix}link4"/>
+      <dynamics damping="0.0" friction="0.0"/>
+    </joint>
+    <link name="${prefix}link4">
       <visual>
         <geometry>
@@ -182,13 +182,13 @@
     </link>
     <!-- Link 5 -->
-    <joint name="joint5" type="revolute">
+    <joint name="${prefix}joint5" type="revolute">
       <axis xyz="0 0 -1" rpy="0 0 0" />
       <limit effort="1000.0" lower="${j5_lower_limit}" upper="${j5_upper_limit}" velocity="${j5_velocity_limit}"/>
       <origin xyz="0 0 ${j4_length}" rpy="0 ${dh_j4_j5_roty} 0" />
-      <parent link="link4"/>
-      <child link="link5"/>
-      <dynamics damping="0.0" friction="0.0"/>
-    </joint>
-    <link name="link5">
+      <parent link="${prefix}link4"/>
+      <child link="${prefix}link5"/>
+      <dynamics damping="0.0" friction="0.0"/>
+    </joint>
+    <link name="${prefix}link5">
       <visual>
         <geometry>
@@ -208,13 +208,13 @@
     </link>
     <!-- Link 6 -->
-    <joint name="joint6" type="revolute">
+    <joint name="${prefix}joint6" type="revolute">
       <axis xyz="0 0 1" rpy="0 0 0" />
       <limit effort="1000.0" lower="${j6_lower_limit}" upper="${j6_upper_limit}" velocity="${j6_velocity_limit}"/>
       <origin xyz="${j5_length} 0 0" rpy="0 ${dh_j5_j6_roty} 0" />
-      <parent link="link5"/>
-      <child link="link6"/>
-      <dynamics damping="0.0" friction="0.0"/>
-    </joint>
-    <link name="link6">
+      <parent link="${prefix}link5"/>
+      <child link="${prefix}link6"/>
+      <dynamics damping="0.0" friction="0.0"/>
+    </joint>
+    <link name="${prefix}link6">
       <visual>
         <geometry>

File: rs_description/urdf/rs080n.urdf.xacro (robot description, xacro)
@@ -3,5 +3,5 @@
   <xacro:include filename="$(find rs_description)/urdf/rs080n_macro.xacro"/>
   <!-- instantiate rs080n -->
-  <xacro:khi_rs080n />
+  <xacro:khi_rs080n prefix="" />
   <!-- Fix rs080n to world -->
   <link name="world"/>
