Commit message: description: add 'prefix' arg to xacro macro.
Allows for prepending a prefix to the name of links and joints, to avoid name clashes between links and joints from other xacro macros in a composite xacro.

File: rs_description/urdf/rs080n_macro.xacro (robot description, xacro)
@@ -1,5 +1,5 @@
 <?xml version="1.0"?>
 <robot xmlns:xacro="http://ros.org/wiki/xacro">
-  <xacro:macro name="khi_rs080n">
+  <xacro:macro name="khi_rs080n" params="prefix">
     <xacro:include filename="$(find rs_description)/urdf/rs.transmission.xacro" />
     <xacro:include filename="$(find rs_description)/urdf/common.gazebo.xacro" />
@@ -60,5 +60,5 @@
     <!-- rs080n start -->
     <!-- Link 0 -->
-    <link name="base_link">
+    <link name="${prefix}base_link">
       <visual>
         <geometry>
@@ -78,13 +78,13 @@
     </link>
     <!-- Link 1 -->
-    <joint name="joint1" type="revolute">
+    <joint name="${prefix}joint1" type="revolute">
       <axis xyz="0 0 -1" rpy="0 0 0" />
       <limit effort="1000.0" lower="${j1_lower_limit}" upper="${j1_upper_limit}" velocity="${j1_velocity_limit}"/>
       <origin xyz="0 0 ${j0_length}" rpy="0 0 0" />
-      <parent link="base_link"/>
-      <child link="link1"/>
-      <dynamics damping="0.0" friction="0.0"/>
-    </joint>
-    <link name="link1">
+      <parent link="${prefix}base_link"/>
+      <child link="${prefix}link1"/>
+      <dynamics damping="0.0" friction="0.0"/>
+    </joint>
+    <link name="${prefix}link1">
       <visual>
         <geometry>
@@ -104,13 +104,13 @@
     </link>
     <!-- Link 2 -->
-    <joint name="joint2" type="revolute">
+    <joint name="${prefix}joint2" type="revolute">
       <axis xyz="0 0 1" rpy="0 0 0" />
       <limit effort="1000.0" lower="${j2_lower_limit}" upper="${j2_upper_limit}" velocity="${j2_velocity_limit}"/>
       <origin xyz="0 ${j1_length} 0" rpy="0 ${dh_j1_j2_roty} 0" />
-      <parent link="link1"/>
-      <child link="link2"/>
-      <dynamics damping="0.0" friction="0.0"/>
-    </joint>
-    <link name="link2">
+      <parent link="${prefix}link1"/>
+      <child link="${prefix}link2"/>
+      <dynamics damping="0.0" friction="0.0"/>
+    </joint>
+    <link name="${prefix}link2">
       <visual>
         <geometry>
@@ -130,13 +130,13 @@
     </link>
     <!-- Link 3 -->
-    <joint name="joint3" type="revolute">
+    <joint name="${prefix}joint3" type="revolute">
       <axis xyz="0 0 -1" rpy="0 0 0" />
       <limit effort="1000.0" lower="${j3_lower_limit}" upper="${j3_upper_limit}" velocity="${j3_velocity_limit}"/>
       <origin xyz="${j2_length} 0 0" rpy="0 0 0" />
-      <parent link="link2"/>
-      <child link="link3"/>
-      <dynamics damping="0.0" friction="0.0"/>
-    </joint>
-    <link name="link3">
+      <parent link="${prefix}link2"/>
+      <child link="${prefix}link3"/>
+      <dynamics damping="0.0" friction="0.0"/>
+    </joint>
+    <link name="${prefix}link3">
       <visual>
         <geometry>
@@ -156,13 +156,13 @@
     </link>
     <!-- Link 4 -->
-    <joint name="joint4" type="revolute">
+    <joint name="${prefix}joint4" type="revolute">
       <axis xyz="0 0 1" rpy="0 0 0" />
       <limit effort="1000.0" lower="${j4_lower_limit}" upper="${j4_upper_limit}" velocity="${j4_velocity_limit}"/>
       <origin xyz="${j3_length} 0 0" rpy="0 ${dh_j3_j4_roty} 0" />
-      <parent link="link3"/>
-      <child link="link4"/>
-      <dynamics damping="0.0" friction="0.0"/>
-    </joint>
-    <link name="link4">
+      <parent link="${prefix}link3"/>
+      <child link="${prefix}link4"/>
+      <dynamics damping="0.0" friction="0.0"/>
+    </joint>
+    <link name="${prefix}link4">
       <visual>
         <geometry>
@@ -182,13 +182,13 @@
     </link>
     <!-- Link 5 -->
-    <joint name="joint5" type="revolute">
+    <joint name="${prefix}joint5" type="revolute">
       <axis xyz="0 0 -1" rpy="0 0 0" />
       <limit effort="1000.0" lower="${j5_lower_limit}" upper="${j5_upper_limit}" velocity="${j5_velocity_limit}"/>
       <origin xyz="0 0 ${j4_length}" rpy="0 ${dh_j4_j5_roty} 0" />
-      <parent link="link4"/>
-      <child link="link5"/>
-      <dynamics damping="0.0" friction="0.0"/>
-    </joint>
-    <link name="link5">
+      <parent link="${prefix}link4"/>
+      <child link="${prefix}link5"/>
+      <dynamics damping="0.0" friction="0.0"/>
+    </joint>
+    <link name="${prefix}link5">
       <visual>
         <geometry>
@@ -208,13 +208,13 @@
     </link>
     <!-- Link 6 -->
-    <joint name="joint6" type="revolute">
+    <joint name="${prefix}joint6" type="revolute">
       <axis xyz="0 0 1" rpy="0 0 0" />
       <limit effort="1000.0" lower="${j6_lower_limit}" upper="${j6_upper_limit}" velocity="${j6_velocity_limit}"/>
       <origin xyz="${j5_length} 0 0" rpy="0 ${dh_j5_j6_roty} 0" />
-      <parent link="link5"/>
-      <child link="link6"/>
-      <dynamics damping="0.0" friction="0.0"/>
-    </joint>
-    <link name="link6">
+      <parent link="${prefix}link5"/>
+      <child link="${prefix}link6"/>
+      <dynamics damping="0.0" friction="0.0"/>
+    </joint>
+    <link name="${prefix}link6">
       <visual>
         <geometry>
