Commit message: description: Jade+ xacro already defines 'pi'.
Indigo is not supported.

File: duaro_description/urdf/duaro_macro.xacro (robot description, xacro)
@@ -3,6 +3,4 @@
   <xacro:macro name="duaro">
     <xacro:include filename="$(find duaro_description)/urdf/duaro.transmission.xacro" />
-    <!-- mathematical value -->
-    <xacro:property name="pi" value="3.14159265359" />
     <!-- DH params -->
     <xacro:property name="dh_j1_j2_transy" value="0.36"/>

File: rs_description/urdf/rs007l_macro.xacro (robot description, xacro)
@@ -4,6 +4,4 @@
     <xacro:include filename="$(find rs_description)/urdf/rs.transmission.xacro" />
     <xacro:include filename="$(find rs_description)/urdf/common.gazebo.xacro" />
-    <!-- mathematics value-->
-    <xacro:property name="pi" value="3.14159265359" />
     <!-- link rviz colors -->
     <material name="White">

File: rs_description/urdf/rs007n_macro.xacro (robot description, xacro)
@@ -4,6 +4,4 @@
     <xacro:include filename="$(find rs_description)/urdf/rs.transmission.xacro" />
     <xacro:include filename="$(find rs_description)/urdf/common.gazebo.xacro" />
-    <!-- mathematics value-->
-    <xacro:property name="pi" value="3.1415" />
     <!-- link rviz colors -->
     <material name="White">

File: rs_description/urdf/rs080n_macro.xacro (robot description, xacro)
@@ -4,6 +4,4 @@
     <xacro:include filename="$(find rs_description)/urdf/rs.transmission.xacro" />
     <xacro:include filename="$(find rs_description)/urdf/common.gazebo.xacro" />
-    <!-- mathematics value-->
-    <xacro:property name="pi" value="3.14159265359" />
     <!-- link rviz colors -->
     <material name="White">

Commit message: description: use 'radians()' support in xacro.

File: duaro_description/urdf/duaro_macro.xacro (robot description, xacro)
@@ -24,25 +24,25 @@
     <xacro:property name="U2_length" value="0.124648"/>
     <!-- joint limits [rad][m] -->
-    <xacro:property name="J1_LOWER_lower_limit" value="${-pi*170/180}"/>
-    <xacro:property name="J1_LOWER_upper_limit" value="${pi*170/180}"/>
-    <xacro:property name="J2_LOWER_lower_limit" value="${-pi*140/180}"/>
-    <xacro:property name="J2_LOWER_upper_limit" value="${pi*140/180}"/>
+    <xacro:property name="J1_LOWER_lower_limit" value="${radians(-170)}"/>
+    <xacro:property name="J1_LOWER_upper_limit" value="${radians( 170)}"/>
+    <xacro:property name="J2_LOWER_lower_limit" value="${radians(-140)}"/>
+    <xacro:property name="J2_LOWER_upper_limit" value="${radians( 140)}"/>
     <xacro:property name="J3_LOWER_lower_limit" value="0"/>
     <xacro:property name="J3_LOWER_upper_limit" value="0.15"/>
-    <xacro:property name="J4_LOWER_lower_limit" value="${-pi*2}"/>
-    <xacro:property name="J4_LOWER_upper_limit" value="${pi*2}"/>
-    <xacro:property name="J1_UPPER_lower_limit" value="${-pi*140/180}"/>
-    <xacro:property name="J1_UPPER_upper_limit" value="${pi*500/180}"/>
-    <xacro:property name="J2_UPPER_lower_limit" value="${-pi*140/180}"/>
-    <xacro:property name="J2_UPPER_upper_limit" value="${pi*140/180}"/>
+    <xacro:property name="J4_LOWER_lower_limit" value="${radians(-360)}"/>
+    <xacro:property name="J4_LOWER_upper_limit" value="${radians( 360)}"/>
+    <xacro:property name="J1_UPPER_lower_limit" value="${radians(-140)}"/>
+    <xacro:property name="J1_UPPER_upper_limit" value="${radians( 500)}"/>
+    <xacro:property name="J2_UPPER_lower_limit" value="${radians(-140)}"/>
+    <xacro:property name="J2_UPPER_upper_limit" value="${radians( 140)}"/>
     <xacro:property name="J3_UPPER_lower_limit" value="0"/>
     <xacro:property name="J3_UPPER_upper_limit" value="0.15"/>
-    <xacro:property name="J4_UPPER_lower_limit" value="${-pi*2}"/>
-    <xacro:property name="J4_UPPER_upper_limit" value="${pi*2}"/>
+    <xacro:property name="J4_UPPER_lower_limit" value="${radians(-360)}"/>
+    <xacro:property name="J4_UPPER_upper_limit" value="${radians( 360)}"/>
     <!-- joint velocity limits [rad/s][m/s]-->
-    <xacro:property name="J1_velocity_limit" value="${pi*240/180}"/>
-    <xacro:property name="J2_velocity_limit" value="${pi*315/180}"/>
+    <xacro:property name="J1_velocity_limit" value="${radians(240)}"/>
+    <xacro:property name="J2_velocity_limit" value="${radians(315)}"/>
     <xacro:property name="J3_velocity_limit" value="0.3"/>
-    <xacro:property name="J4_velocity_limit" value="${pi*600/180}"/>
+    <xacro:property name="J4_velocity_limit" value="${radians(600)}"/>
     <!-- link rviz color-->
     <material name="Light_blue">

File: rs_description/urdf/rs007l_macro.xacro (robot description, xacro)
@@ -12,8 +12,8 @@
     </material>
     <!-- DH parameters -->
-    <xacro:property name="dh_j1_j2_roty" value="-${pi/2}"/>
-    <xacro:property name="dh_j3_j4_roty" value="${pi/2}"/>
-    <xacro:property name="dh_j4_j5_roty" value="-${pi/2}"/>
-    <xacro:property name="dh_j5_j6_roty" value="${pi/2}"/>
+    <xacro:property name="dh_j1_j2_roty" value="${radians(-90)}"/>
+    <xacro:property name="dh_j3_j4_roty" value="${radians( 90)}"/>
+    <xacro:property name="dh_j4_j5_roty" value="${radians(-90)}"/>
+    <xacro:property name="dh_j5_j6_roty" value="${radians( 90)}"/>
     <!-- link mass [kg] -->
     <xacro:property name="j0_mass" value="11"/>
@@ -32,23 +32,23 @@
     <xacro:property name="j5_length" value="0.078"/>
     <!-- joint limits [rad] -->
-    <xacro:property name="j1_lower_limit" value="${-pi}"/>
-    <xacro:property name="j1_upper_limit" value="${pi}"/>
-    <xacro:property name="j2_lower_limit" value="${-pi*135/180}"/>
-    <xacro:property name="j2_upper_limit" value="${pi*135/180}"/>
-    <xacro:property name="j3_lower_limit" value="${-pi*157/180}"/>
-    <xacro:property name="j3_upper_limit" value="${pi*157/180}"/>
-    <xacro:property name="j4_lower_limit" value="${-pi*200/180}"/>
-    <xacro:property name="j4_upper_limit" value="${pi*200/180}"/>
-    <xacro:property name="j5_lower_limit" value="${-pi*125/180}"/>
-    <xacro:property name="j5_upper_limit" value="${pi*125/180}"/>
-    <xacro:property name="j6_lower_limit" value="${-2*pi}"/>
-    <xacro:property name="j6_upper_limit" value="${2*pi}"/>
+    <xacro:property name="j1_lower_limit" value="${radians(-180)}"/>
+    <xacro:property name="j1_upper_limit" value="${radians( 180)}"/>
+    <xacro:property name="j2_lower_limit" value="${radians(-135)}"/>
+    <xacro:property name="j2_upper_limit" value="${radians( 135)}"/>
+    <xacro:property name="j3_lower_limit" value="${radians(-157)}"/>
+    <xacro:property name="j3_upper_limit" value="${radians( 157)}"/>
+    <xacro:property name="j4_lower_limit" value="${radians(-200)}"/>
+    <xacro:property name="j4_upper_limit" value="${radians( 200)}"/>
+    <xacro:property name="j5_lower_limit" value="${radians(-125)}"/>
+    <xacro:property name="j5_upper_limit" value="${radians( 125)}"/>
+    <xacro:property name="j6_lower_limit" value="${radians(-360)}"/>
+    <xacro:property name="j6_upper_limit" value="${radians( 360)}"/>
     <!-- joint verocity limits [rad/s] -->
-    <xacro:property name="j1_velocity_limit" value="${pi*370/180}"/>
-    <xacro:property name="j2_velocity_limit" value="${pi*310/180}"/>
-    <xacro:property name="j3_velocity_limit" value="${pi*410/180}"/>
-    <xacro:property name="j4_velocity_limit" value="${pi*550/180}"/>
-    <xacro:property name="j5_velocity_limit" value="${pi*550/180}"/>
-    <xacro:property name="j6_velocity_limit" value="${pi*1000/180}"/>
+    <xacro:property name="j1_velocity_limit" value="${radians( 370)}"/>
+    <xacro:property name="j2_velocity_limit" value="${radians( 310)}"/>
+    <xacro:property name="j3_velocity_limit" value="${radians( 410)}"/>
+    <xacro:property name="j4_velocity_limit" value="${radians( 550)}"/>
+    <xacro:property name="j5_velocity_limit" value="${radians( 550)}"/>
+    <xacro:property name="j6_velocity_limit" value="${radians(1000)}"/>
     <!-- link inertial(TODO : set correct link inertial )-->
     <xacro:macro name="default_inertial" params="mass">

File: rs_description/urdf/rs007n_macro.xacro (robot description, xacro)
@@ -12,8 +12,8 @@
     </material>
     <!-- DH parameters -->
-    <xacro:property name="dh_j1_j2_roty" value="-${pi/2}"/>
-    <xacro:property name="dh_j3_j4_roty" value="${pi/2}"/>
-    <xacro:property name="dh_j4_j5_roty" value="-${pi/2}"/>
-    <xacro:property name="dh_j5_j6_roty" value="${pi/2}"/>
+    <xacro:property name="dh_j1_j2_roty" value="${radians(-90)}"/>
+    <xacro:property name="dh_j3_j4_roty" value="${radians( 90)}"/>
+    <xacro:property name="dh_j4_j5_roty" value="${radians(-90)}"/>
+    <xacro:property name="dh_j5_j6_roty" value="${radians( 90)}"/>
     <!-- link mass [kg] -->
     <xacro:property name="j0_mass" value="11"/>
@@ -32,23 +32,23 @@
     <xacro:property name="j5_length" value="0.078"/>
     <!-- joint limits [rad] -->
-    <xacro:property name="j1_lower_limit" value="${-pi}"/>
-    <xacro:property name="j1_upper_limit" value="${pi}"/>
-    <xacro:property name="j2_lower_limit" value="${-pi*135/180}"/>
-    <xacro:property name="j2_upper_limit" value="${pi*135/180}"/>
-    <xacro:property name="j3_lower_limit" value="${-pi*155/180}"/>
-    <xacro:property name="j3_upper_limit" value="${pi*155/180}"/>
-    <xacro:property name="j4_lower_limit" value="${-pi*200/180}"/>
-    <xacro:property name="j4_upper_limit" value="${pi*200/180}"/>
-    <xacro:property name="j5_lower_limit" value="${-pi*125/180}"/>
-    <xacro:property name="j5_upper_limit" value="${pi*125/180}"/>
-    <xacro:property name="j6_lower_limit" value="${-2*pi}"/>
-    <xacro:property name="j6_upper_limit" value="${2*pi}"/>
+    <xacro:property name="j1_lower_limit" value="${radians(-180)}"/>
+    <xacro:property name="j1_upper_limit" value="${radians( 180)}"/>
+    <xacro:property name="j2_lower_limit" value="${radians(-135)}"/>
+    <xacro:property name="j2_upper_limit" value="${radians( 135)}"/>
+    <xacro:property name="j3_lower_limit" value="${radians(-155)}"/>
+    <xacro:property name="j3_upper_limit" value="${radians( 155)}"/>
+    <xacro:property name="j4_lower_limit" value="${radians(-200)}"/>
+    <xacro:property name="j4_upper_limit" value="${radians( 200)}"/>
+    <xacro:property name="j5_lower_limit" value="${radians(-125)}"/>
+    <xacro:property name="j5_upper_limit" value="${radians( 125)}"/>
+    <xacro:property name="j6_lower_limit" value="${radians(-360)}"/>
+    <xacro:property name="j6_upper_limit" value="${radians( 360)}"/>
     <!-- joint verocity limits [rad/s] -->
-    <xacro:property name="j1_velocity_limit" value="${pi*470/180}"/>
-    <xacro:property name="j2_velocity_limit" value="${pi*380/180}"/>
-    <xacro:property name="j3_velocity_limit" value="${pi*520/180}"/>
-    <xacro:property name="j4_velocity_limit" value="${pi*550/180}"/>
-    <xacro:property name="j5_velocity_limit" value="${pi*550/180}"/>
-    <xacro:property name="j6_velocity_limit" value="${pi*1000/180}"/>
+    <xacro:property name="j1_velocity_limit" value="${radians( 470)}"/>
+    <xacro:property name="j2_velocity_limit" value="${radians( 380)}"/>
+    <xacro:property name="j3_velocity_limit" value="${radians( 520)}"/>
+    <xacro:property name="j4_velocity_limit" value="${radians( 550)}"/>
+    <xacro:property name="j5_velocity_limit" value="${radians( 550)}"/>
+    <xacro:property name="j6_velocity_limit" value="${radians(1000)}"/>
     <!-- link inertial(TODO : set correct link inertial )-->
     <xacro:macro name="default_inertial" params="mass">

File: rs_description/urdf/rs080n_macro.xacro (robot description, xacro)
@@ -12,8 +12,8 @@
     </material>
     <!-- DH parameters -->
-    <xacro:property name="dh_j1_j2_roty" value="-${pi/2}"/>
-    <xacro:property name="dh_j3_j4_roty" value="${pi/2}"/>
-    <xacro:property name="dh_j4_j5_roty" value="-${pi/2}"/>
-    <xacro:property name="dh_j5_j6_roty" value="${pi/2}"/>
+    <xacro:property name="dh_j1_j2_roty" value="${radians(-90)}"/>
+    <xacro:property name="dh_j3_j4_roty" value="${radians( 90)}"/>
+    <xacro:property name="dh_j4_j5_roty" value="${radians(-90)}"/>
+    <xacro:property name="dh_j5_j6_roty" value="${radians( 90)}"/>
     <!-- link mass [kg] -->
     <xacro:property name="j0_mass" value="200"/> <!-- TO-DO -->
@@ -32,23 +32,23 @@
     <xacro:property name="j5_length" value="0.165"/>
     <!-- joint limits [rad] -->
-    <xacro:property name="j1_lower_limit" value="${-pi}"/>
-    <xacro:property name="j1_upper_limit" value="${pi}"/>
-    <xacro:property name="j2_lower_limit" value="${-pi*105/180}"/>
-    <xacro:property name="j2_upper_limit" value="${pi*140/180}"/>
-    <xacro:property name="j3_lower_limit" value="${-pi*155/180}"/>
-    <xacro:property name="j3_upper_limit" value="${pi*135/180}"/>
-    <xacro:property name="j4_lower_limit" value="${-pi*360/180}"/>
-    <xacro:property name="j4_upper_limit" value="${pi*360/180}"/>
-    <xacro:property name="j5_lower_limit" value="${-pi*145/180}"/>
-    <xacro:property name="j5_upper_limit" value="${pi*145/180}"/>
-    <xacro:property name="j6_lower_limit" value="${-pi*360/180}"/>
-    <xacro:property name="j6_upper_limit" value="${pi*360/180}"/>
+    <xacro:property name="j1_lower_limit" value="${radians(-180)}"/>
+    <xacro:property name="j1_upper_limit" value="${radians( 180)}"/>
+    <xacro:property name="j2_lower_limit" value="${radians(-105)}"/>
+    <xacro:property name="j2_upper_limit" value="${radians( 150)}"/>
+    <xacro:property name="j3_lower_limit" value="${radians(-155)}"/>
+    <xacro:property name="j3_upper_limit" value="${radians( 135)}"/>
+    <xacro:property name="j4_lower_limit" value="${radians(-360)}"/>
+    <xacro:property name="j4_upper_limit" value="${radians( 360)}"/>
+    <xacro:property name="j5_lower_limit" value="${radians(-145)}"/>
+    <xacro:property name="j5_upper_limit" value="${radians( 145)}"/>
+    <xacro:property name="j6_lower_limit" value="${radians(-360)}"/>
+    <xacro:property name="j6_upper_limit" value="${radians( 360)}"/>
     <!-- joint velocity limits [rad/s] -->
-    <xacro:property name="j1_velocity_limit" value="${pi*180/180}"/>
-    <xacro:property name="j2_velocity_limit" value="${pi*180/180}"/>
-    <xacro:property name="j3_velocity_limit" value="${pi*160/180}"/>
-    <xacro:property name="j4_velocity_limit" value="${pi*185/180}"/>
-    <xacro:property name="j5_velocity_limit" value="${pi*165/180}"/>
-    <xacro:property name="j6_velocity_limit" value="${pi*280/180}"/>
+    <xacro:property name="j1_velocity_limit" value="${radians(180)}"/>
+    <xacro:property name="j2_velocity_limit" value="${radians(180)}"/>
+    <xacro:property name="j3_velocity_limit" value="${radians(160)}"/>
+    <xacro:property name="j4_velocity_limit" value="${radians(185)}"/>
+    <xacro:property name="j5_velocity_limit" value="${radians(165)}"/>
+    <xacro:property name="j6_velocity_limit" value="${radians(280)}"/>
     <!-- link inertial(TODO : set correct link inertial )-->
     <xacro:macro name="default_inertial" params="mass">
