Commit message: rs_desc: add 'base' frame.
This maps between ROS and KHI coordinate origins (ie: world frame).

Note: Kawasaki robots have Y+ 'forward'. This frame compensates for that by rotating -90 degrees around Z.

File: rs_description/urdf/rs007l_macro.xacro (robot description, xacro)
@@ -233,4 +233,11 @@
       <xacro:default_inertial mass="${j6_mass}"/>
     </link>
+    <!-- ROS-Industrial 'base' frame: base_link to Kawasaki Base Coordinates transform -->
+    <link name="${prefix}base" />
+    <joint name="${prefix}base_link-base" type="fixed">
+      <origin xyz="0 0 ${j0_length}" rpy="0 0 ${radians(-90)}"/>
+      <parent link="${prefix}base_link"/>
+      <child link="${prefix}base"/>
+    </joint>
   </xacro:macro>
 </robot>

Commit message: rs_desc: add 'flange' frame.
Easy attachment point for EEF models (ROS has X+ 'forward').

File: rs_description/urdf/rs007l_macro.xacro (robot description, xacro)
@@ -240,4 +240,11 @@
       <child link="${prefix}base"/>
     </joint>
+    <!-- ROS-Industrial 'flange' frame: attachment point for EEF models -->
+    <link name="${prefix}flange" />
+    <joint name="${prefix}link6-flange" type="fixed">
+      <origin xyz="0 0 0" rpy="0 0 0" />
+      <parent link="${prefix}link6" />
+      <child link="${prefix}flange" />
+    </joint>
   </xacro:macro>
 </robot>

Commit message: rs_desc: add 'tool0' frame.
Aligns with an all-zeros TOOL frame on Kawasaki controller.

Transforms between 'base' and 'tool0' should be identical to those reported by the Kawasaki controller.

File: rs_description/urdf/rs007l_macro.xacro (robot description, xacro)
@@ -247,4 +247,11 @@
       <child link="${prefix}flange" />
     </joint>
+    <!-- ROS-Industrial 'tool0' frame: all-zeros tool frame -->
+    <link name="${prefix}tool0" />
+    <joint name="${prefix}link6-tool0" type="fixed">
+      <origin xyz="0 0 0" rpy="0 0 ${radians(-90)}" />
+      <parent link="${prefix}link6" />
+      <child link="${prefix}tool0" />
+    </joint>
   </xacro:macro>
 </robot>
